Commit message: Sanity check: lab 9

File: src/robot_control/urdf/su_robot.urdf (robot description, URDF)
Before this commit: robot origins, 10 links, 9 joints
Links:
- added link camera; visual cylinder length=0.01 radius=0.07
Joints:
- joint base_to_back_left_leg: axis 1 0 0 -> 0 1 0; origin xyz=-0.16 0.26 0.0 rpy=0 0 1.57075 -> xyz=0.16 0.26 0.0 rpy=0 0 0
- joint base_to_back_right_leg: axis 1 0 0 -> 0 1 0; origin xyz=-0.16 -0.26 0.0 rpy=0 0 1.57075 -> xyz=0.16 -0.26 0.0 rpy=0 0 0
- joint base_to_front_left_leg: axis 1 0 0 -> 0 1 0; origin xyz=0.16 0.26 0.0 rpy=0 0 1.57075 -> xyz=-0.16 0.26 0.0 rpy=0 0 0
- joint base_to_front_right_leg: axis 1 0 0 -> 0 1 0; origin xyz=0.16 -0.26 0.0 rpy=0 0 1.57075 -> xyz=-0.16 -0.26 0.0 rpy=0 0 3.14159
